File: Forklift_prototip_karti.kicad_sch (KiCad schematic)
At the start: 25 parts, among them J10 Mini360, J11 Barrel_Jack_Switch, J6 Conn_01x22_Pin, J7 Conn_01x22_Pin, U1 ESP32-S3-DEVKITC-1-N8R2, U2 PCF8563T, Y1 32.768 KHz

Commit message: Add files via upload
Connections:
- net IO45: now also S-K-B1.1 (Pin_1); no longer S-K-B1.2 (Pin_2)
- net IO48: now also S-K-B1.2 (Pin_2); no longer S-K-B1.1 (Pin_1)
Changed lines of the file:
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@@
 		)
 	)
-	(label "IO45"
+	(label "IO48"
 		(at 207.01 34.29 0)
 		(effects
@@
 		)
 	)
-	(label "IO48"
+	(label "IO45"
 		(at 207.01 31.75 0)
 		(effects
